Commit message: Add ros2_robotiq_gripper as a submodule

File: src/combined_robot_description/urdf/bmw_ur5_gripper_combined.urdf.xacro (robot description, xacro)
@@ -5,4 +5,5 @@
   <xacro:bmw_car prefix="bmw_"/>
   <xacro:include filename="/home/christopher/warde/src/Universal_Robots_ROS2_Description/urdf/ur_macro.xacro"/>
+  <xacro:include filename="/home/christopher/warde/src/ros2_robotiq_gripper/robotiq_description/urdf/robotiq_2f_140_macro.urdf.xacro"/>
   <!-- instantiate a UR5, parented to the BMW’s chassis link, 0.3 m above it -->
   <xacro:ur_robot
@@ -20,3 +21,11 @@
     <origin xyz="-0.18 0 0.225" rpy="0 0 0"/>
     </xacro:ur_robot>
+  <xacro:robotiq_gripper
+    name="robotiq_2f_140"
+    prefix="gripper_"
+    parent="ur5_wrist_3_link"
+    use_fake_hardware="true"
+    include_ros2_control="true">
+    <origin xyz="0 0 0.15" rpy="0 0 0"/>
+    </xacro:robotiq_gripper>
 </robot>
